File: 4HP_555_eg.brd (EAGLE design)
At the start: 101.9 x 19.7 mm, 49 parts, among them IC1 IC_555-SOIC8, Q1 MMBT5088, Q2 MMBT5088, Q3 MMBT5088, Q4 MMBT5088

Commit message: 4HP 555 ADSR EG
LM555 ADSR Envelope Generator
Parts:
- C1, C2: value (none) -> 10uF
Changed lines of the file:
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@@
 <?xml version="1.0" encoding="utf-8"?>
 <!DOCTYPE eagle SYSTEM "eagle.dtd">
-<eagle version="7.5.0">
+<eagle version="8.1.1">
 <drawing>
 <settings>
@@
 <element name="R10" library="SparkFun-Passives" package="0603-RES" value="1M" x="16.8275" y="10.795"/>
 <element name="R11" library="SparkFun-Passives" package="0603-RES" value="1M" x="16.8275" y="13.97" rot="R180"/>
-<element name="C1" library="capacitors-elec" package="050_020_1" value="" x="68.58" y="4.445" rot="R90"/>
-<element name="C2" library="capacitors-elec" package="050_020_1" value="" x="68.58" y="16.1925" rot="R90"/>
+<element name="C1" library="capacitors-elec" package="050_020_1" value="10uF" x="68.58" y="4.445" rot="R90"/>
+<element name="C2" library="capacitors-elec" package="050_020_1" value="10uF" x="68.58" y="16.1925" rot="R90"/>
 <element name="R12" library="SparkFun-Passives" package="0603-RES" value="22K" x="20.955" y="12.7"/>
 <element name="R13" library="SparkFun-Passives" package="0603-RES" value="22K" x="24.13" y="12.7" rot="R180"/>
